File: 6g_att/6g_att/6g_att.kicad_pcb (KiCad board)
At the start: 2 copper layers, 100 x 100 mm, 150 parts, among them J1 Conn_Coaxial, J2 Conn_Coaxial, J3 Conn_Coaxial, J4 Conn_Coaxial, J5 Conn_Coaxial, J6 Conn_Coaxial, J7 Conn_Coaxial, J8 Conn_Coaxial

Commit message: connected touch pads
Parts:
- turned R1 to -90 degrees
- turned R104 to -90 degrees
- turned R105 to 90 degrees
- turned R106 to -90 degrees
- turned R107 to -90 degrees
- turned R108 to 90 degrees
- turned R109 to -90 degrees
- turned R110 to 90 degrees
- turned R119 to 90 degrees
- turned R120 to 90 degrees
- turned R121 to -90 degrees
- turned R124 to -90 degrees
- turned R127 to 90 degrees
- turned R128 to 90 degrees
- turned R129 to -90 degrees
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
Commit message: before stitch
Parts:
- J3, J4, J5, J8, R12, R17, R25, R28, R37, R47, R48, R8: moved to B.Cu
- moved J8 174.1 mm to (175.0, 149.0), turned to -90 degrees
- moved J5 158.5 mm to (173.9, 53.2), turned to 90 degrees
- moved J3 144.1 mm to (102.6, 149.0), turned to -90 degrees
- moved R138 130.1 mm to (98.3, 141.2), turned to 90 degrees
- moved R137 125.4 mm to (98.3, 138.4), turned to -90 degrees
- moved R66 123.9 mm to (165.8, 141.2), turned to 90 degrees
- moved R141 120.8 mm to (98.3, 135.5), turned to 90 degrees
- moved R134 119.3 mm to (101.7, 137.0), turned to 0 degrees
- moved R65 119.0 mm to (165.8, 138.4), turned to -90 degrees
- moved J2 116.8 mm to (91.0, 114.3), turned to 180 degrees
- moved R142 116.3 mm to (98.3, 132.7), turned to -90 degrees
- moved R133 116.2 mm to (104.5, 137.0), turned to 180 degrees
- moved R128 115.3 mm to (107.8, 138.4), turned to -90 degrees
- moved R75 114.2 mm to (165.8, 135.5), turned to 90 degrees
- moved R12 113.8 mm to (134.3, 102.8), turned to 90 degrees
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Routing:
- net Net-(J3-In): track 0.00 -> 116.5 mm
- net Net-(J4-In): track 0.00 -> 66.4 mm
- net Net-(J5-In): track 0.00 -> 65.8 mm
- net Net-(R62-Pad1): track 0.00 -> 53.5 mm
- net Net-(R65-Pad1): track 0.00 -> 44.6 mm
- net Net-(J2-In): track 0.00 -> 11.6 mm
- net Net-(J7-In): track 0.00 -> 11.6 mm
- net Net-(J1-In): track 0.01 -> 9.25 mm
- net Net-(J6-In): track 0.00 -> 9.17 mm
- net Net-(R35-Pad2): track 0.00 -> 4.83 mm
- net Net-(R23-Pad2): track 0.00 -> 4.83 mm
- net Net-(R126-Pad1): track 0.00 -> 4.83 mm
- net Net-(R118-Pad1): track 0.00 -> 4.83 mm
- net Net-(R11-Pad2): track 0.00 -> 4.83 mm
- net Net-(R83-Pad1): track 0.00 -> 4.82 mm
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- added copper zone on B.Cu, net GND
- added copper zone on F.Cu, net GND
