File: 6g_att/6g_att/6g_att.kicad_pcb (KiCad board)
At the start: 2 copper layers, 100 x 100 mm, 150 parts, among them J1 Conn_Coaxial, J2 Conn_Coaxial, J3 Conn_Coaxial, J4 Conn_Coaxial, J5 Conn_Coaxial, J6 Conn_Coaxial, J7 Conn_Coaxial, J8 Conn_Coaxial

Commit message: add logo
Other:
- board text added: "zxkmm DC-6GHz 20dB + 10dB fine tune +10dBm safer for SA zxkmm.com JLCJLCJLCJLC"
- board text added: "███╗ ███╗ █████╗ ██╗ ██╗ ██╗ ██████╗ ██╗ ██╗ █████╗ ████████╗████████╗ ████╗ ████║██╔══██╗╚██╗██╔╝ ███║██╔═████╗██║ ██║ ██╔══██╗╚══██╔══╝╚══██╔══╝ ██╔████╔██║███████║ ╚███╔╝ ╚██║██║██╔██║██║ █╗ ██║ ███████║ ██║ ██║ ██║╚██╔╝██║██╔══██║ ██╔██╗ ██║████╔╝██║██║███╗██║ ██╔══██║ ██║ ██║ ██║ ╚═╝ ██║██║ ██║██╔╝ ██╗ ██║╚██████╔╝╚███╔███╔╝ ██║ ██║ ██║ ██║ ╚═╝ ╚═╝╚═╝ ╚═╝╚═╝ ╚═╝ ╚═╝ ╚═════╝ ╚══╝╚══╝ ╚═╝ ╚═╝ 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"
- board text added: "██████╗ ██████╗ ██╗ ██╗ ██████╗ ██████╗ ██████╗ ╚════██╗██╔═████╗ ██╔╝███║██╔═████╗ ██╔══██╗██╔══██╗ █████╔╝██║██╔██║ ██╔╝ ╚██║██║██╔██║ ██║ ██║██████╔╝ ██╔═══╝ ████╔╝██║ ██╔╝ ██║████╔╝██║ ██║ ██║██╔══██╗ ███████╗╚██████╔╝██╔╝ ██║╚██████╔╝ ██████╔╝██████╔╝ ╚══════╝ ╚═════╝ ╚═╝ ╚═╝ ╚═════╝ ╚═════╝ ╚═════╝"
- board text added: "███████╗██╗ ██╗██╗ ██╗███╗ ███╗███╗ ███╗ ╚══███╔╝╚██╗██╔╝██║ ██╔╝████╗ ████║████╗ ████║ ███╔╝ ╚███╔╝ █████╔╝ ██╔████╔██║██╔████╔██║ ███╔╝ ██╔██╗ ██╔═██╗ ██║╚██╔╝██║██║╚██╔╝██║ ███████╗██╔╝ ██╗██║ ██╗██║ ╚═╝ ██║██║ ╚═╝ ██║ ╚══════╝╚═╝ ╚═╝╚═╝ ╚═╝╚═╝ ╚═╝╚═╝ ╚═╝"
